File: kicad/eel_head_pcbs_assembly/eel_esp32_switch_host_board_v02/eel_esp32_switch_host_board_v02.kicad_sch (KiCad schematic)
At the start: 13 parts, among them J1 Lipo back, J2 motor driver, J3 ELRS RX, J4 Noods front, J5 RGB_DATA, J6 Lipo front, J7 Noods back, Q1 BC817, SW1 SW_Push_DPDT, U1 XIAO-ESP32C3

Commit message: update Kicad project (probably nothing)
Other:
- company: (none) -> Adriaan Wormgoor (http://www.adriaanwormgoor.nl)
- title: (none) -> Haribo Kimchi Eel mainboard
Changed lines of the file:
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@@
 (kicad_sch
-	(version 20231120)
+	(version 20250114)
 	(generator "eeschema")
-	(generator_version "8.0")
+	(generator_version "9.0")
 	(paper "A4")
+	(title_block
+		(title "Haribo Kimchi Eel mainboard")
+		(date "2024-02-18")
+		(company "Adriaan Wormgoor (http://www.adriaanwormgoor.nl)")
+	)
+	(text "PADS FACING BACK"
+		(exclude_from_sim no)
+		(at 76.581 80.899 0)
+		(effects
+			(font
+				(size 1.27 1.27)
+			)
+			(justify left bottom)
+		)
+	)
+	(text "PADS FACING FRONT"
+		(exclude_from_sim no)
+		(at 22.098 80.518 0)
+		(effects
+			(font
+				(size 1.27 1.27)
+			)
+			(justify left bottom)
+		)
+	)
 	(junction
 		(at 94.615 90.043)
@@
 			(width 0)
 			(type default)
-		)
-	)
-	(text "PADS FACING BACK"
-		(exclude_from_sim no)
-		(at 76.581 80.899 0)
-		(effects
-			(font
-				(size 1.27 1.27)
-			)
-			(justify left bottom)
-		)
-	)
-	(text "PADS FACING FRONT"
-		(exclude_from_sim no)
-		(at 22.098 80.518 0)
-		(effects
-			(font
-				(size 1.27 1.27)
-			)
-			(justify left bottom)
 		)
 	)
@@
 		)
 	)
+	(embedded_fonts no)
 )
