File: kicad/Adafruit_Feather_M4_Express_breakout_board/Adafruit_Feather_M4_Express_breakout_board.kicad_pcb (KiCad board)
At the start: 2 copper layers, 51.9 x 24.1 mm, 14 parts, among them J1 Conn_01x03_Socket, J2 Conn_01x03_Socket, J3 Conn_01x03_Socket, J4 Conn_01x03_Socket, J5 Conn_01x03_Socket

Commit message: minor label edits to the schematic
Connections:
- net A0_DAC_THROTTLE renamed A1_DAC_THROTTLE
- net A1_DAC_YAW renamed A0_DAC_YAW
Changed lines of the file:
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@@
 	(net 13 "unconnected-(A1-~{RESET}-Pad1)")
 	(net 14 "unconnected-(A1-D13-Pad25)")
-	(net 15 "A1_DAC_YAW")
+	(net 15 "A1_DAC_THROTTLE")
 	(net 16 "unconnected-(A1-MISO{slash}D22-Pad13)")
 	(net 17 "unconnected-(A1-SCK{slash}D24-Pad11)")
@@
 	(net 23 "unconnected-(A1-USB-Pad26)")
 	(net 24 "D1_PWM_AUX2")
-	(net 25 "A0_DAC_THROTTLE")
+	(net 25 "A0_DAC_YAW")
 	(net 26 "unconnected-(A1-SCL{slash}D21-Pad18)")
 	(net 27 "unconnected-(J1-Pin_3-Pad3)")
@@
 			(layers "F.Cu" "F.Mask" "F.Paste")
 			(roundrect_rratio 0.25)
-			(net 15 "A1_DAC_YAW")
+			(net 25 "A0_DAC_YAW")
 			(pinfunction "Pin_1")
 			(pintype "passive")
@@
 			(layers "F.Cu" "F.Mask" "F.Paste")
 			(roundrect_rratio 0.25)
-			(net 25 "A0_DAC_THROTTLE")
+			(net 15 "A1_DAC_THROTTLE")
 			(pinfunction "Pin_1")
 			(pintype "passive")
@@
 			(layers "*.Cu" "*.Mask")
 			(remove_unused_layers no)
-			(net 15 "A1_DAC_YAW")
+			(net 25 "A0_DAC_YAW")
 			(pinfunction "DAC0/A0")
 			(pintype "bidirectional")
@@
 			(layers "*.Cu" "*.Mask")
 			(remove_unused_layers no)
-			(net 25 "A0_DAC_THROTTLE")
+			(net 15 "A1_DAC_THROTTLE")
 			(pinfunction "DAC1/A1")
 			(pintype "bidirectional")
@@
 	)
 	(segment
-		(start 139.176 99.679)
-		(end 139.176 95.449)
-		(width 0.25)
-		(layer "F.Cu")
-		(net 15)
-	)
-	(segment
-		(start 139.192 100.838)
-		(end 139.192 99.695)
-		(width 0.25)
-		(layer "F.Cu")
-		(net 15)
-	)
-	(segment
-		(start 139.192 99.695)
-		(end 139.176 99.679)
+		(start 126.349 100.965)
+		(end 126.349 95.449)
 		(width 0.25)
 		(layer "F.Cu")
@@
 	)
 	(via
-		(at 139.192 100.838)
+		(at 126.349 100.965)
 		(size 0.8)
 		(drill 0.4)
@@
 	)
 	(segment
-		(start 147.828 102.235)
-		(end 152.527 106.934)
+		(start 149.987 105.587)
+		(end 149.987 106.934)
 		(width 0.25)
 		(layer "B.Cu")
@@
 	)
 	(segment
-		(start 140.335 102.235)
-		(end 147.828 102.235)
+		(start 147.27 102.87)
+		(end 149.987 105.587)
 		(width 0.25)
 		(layer "B.Cu")
@@
 	)
 	(segment
-		(start 139.192 101.092)
-		(end 140.335 102.235)
+		(start 126.349 101.584)
+		(end 127.635 102.87)
 		(width 0.25)
 		(layer "B.Cu")
@@
 	)
 	(segment
-		(start 139.192 100.838)
-		(end 139.192 101.092)
+		(start 126.349 100.965)
+		(end 126.349 101.584)
+		(width 0.25)
+		(layer "B.Cu")
+		(net 15)
+	)
+	(segment
+		(start 127.635 102.87)
+		(end 147.27 102.87)
 		(width 0.25)
 		(layer "B.Cu")
@@
 	)
 	(segment
-		(start 126.349 100.965)
-		(end 126.349 95.449)
+		(start 139.176 99.679)
+		(end 139.176 95.449)
 		(width 0.25)
 		(layer "F.Cu")
 		(net 25)
 	)
-	(via
-		(at 126.349 100.965)
-		(size 0.8)
-		(drill 0.4)
-		(layers "F.Cu" "B.Cu")
+	(segment
+		(start 139.192 100.838)
+		(end 139.192 99.695)
+		(width 0.25)
+		(layer "F.Cu")
 		(net 25)
 	)
 	(segment
-		(start 149.987 105.587)
-		(end 149.987 106.934)
+		(start 139.192 99.695)
+		(end 139.176 99.679)
 		(width 0.25)
-		(layer "B.Cu")
+		(layer "F.Cu")
+		(net 25)
+	)
+	(via
+		(at 139.192 100.838)
+		(size 0.8)
+		(drill 0.4)
+		(layers "F.Cu" "B.Cu")
 		(net 25)
 	)
 	(segment
-		(start 147.27 102.87)
-		(end 149.987 105.587)
+		(start 147.828 102.235)
+		(end 152.527 106.934)
 		(width 0.25)
 		(layer "B.Cu")
@@
 	)
 	(segment
-		(start 126.349 101.584)
-		(end 127.635 102.87)
+		(start 140.335 102.235)
+		(end 147.828 102.235)
 		(width 0.25)
 		(layer "B.Cu")
@@
 	)
 	(segment
-		(start 126.349 100.965)
-		(end 126.349 101.584)
+		(start 139.192 101.092)
+		(end 140.335 102.235)
 		(width 0.25)
 		(layer "B.Cu")
@@
 	)
 	(segment
-		(start 127.635 102.87)
-		(end 147.27 102.87)
+		(start 139.192 100.838)
+		(end 139.192 101.092)
 		(width 0.25)
 		(layer "B.Cu")
